File: LI600 SWITCH.kicad_sch (KiCad schematic)
At the start: 29 parts, among them J1 sub_D_25, J2 sub_D_25, J3 Conn_02x25_Odd_Even, J4 Conn_01x05_P2.54mm_pinheader_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

Commit message: version 19/12/2024
Signed-off-by: TEST-BANC <TEST-BANC@DOMOMICRON.LOCAL>
Parts:
- removed J2: sub_D_25, Omiconnecteur:sub_D_25, symbol Omiconnecteur:sub_D_25
- removed J3: Conn_02x25_Odd_Even, Omiconnecteur:PinHeader_2x25_P2.54mm_V_omi, symbol Omiconnecteur:Conn_02x25_Odd_Even_omi
- removed J4: Conn_01x05_P2.54mm_pinheader_vertical, Omiconnecteur:PinHeader_1x05_P2.54mm_V_omi, symbol Omiconnecteur:Conn_01x05_P2.54mm_pinheader_vertical
- added J2: Conn_02x25_Odd_Even, Omiconnecteur:PinHeader_2x25_P2.54mm_V_omi, symbol Omiconnecteur:Conn_02x25_Odd_Even_omi
- added J3: Conn_01x05_P2.54mm_pinheader_vertical, Omiconnecteur:PinHeader_1x05_P2.54mm_V_omi, symbol Omiconnecteur:Conn_01x05_P2.54mm_pinheader_vertical
- added J4: sub_D_25, Omiconnecteur:sub_D_25, symbol Omiconnecteur:sub_D_25
Connections:
- net at J1.1, Terre1.1 (Pin_1): now also J2.1 (Pin_1)
- net at IDC-1+IFC-1.1 (Pin_1), J1.16: now also J2.11 (Pin_11)
- net at GNDMoteur2.1 (Pin_1), J1.6: now also J2.21 (Pin_21); no longer J1.26, J1.27
- net at GNDMoteur1.1 (Pin_1), J1.7: now also J2.25 (Pin_25)
- net at J1.4, VMoteur2.1 (Pin_1): now also J2.13 (Pin_13)
- net at GNDLASER1.1 (Pin_1), J1.17: now also J2.15 (Pin_15)
- net at J1.5, VMoteur3.1 (Pin_1): now also J2.17 (Pin_17)
- net at +5VLASER1.1 (Pin_1), J1.18: now also J2.19 (Pin_19)
- net at J1.19, SwitchOptique2.1 (Pin_1): now also J2.23 (Pin_23)
- net at J1.20, SwitchOptique3.1 (Pin_1): now also J2.27 (Pin_27)
- net at GNDMoteur3.1 (Pin_1), J1.8: now also J2.29 (Pin_29)
- net at IDC-1.1 (Pin_1), J1.14: now also J2.3 (Pin_3)
- net at +5VREGLE1.1 (Pin_1), J1.21: now also J2.31 (Pin_31)
- net at J1.9, SwitchOptique1.1 (Pin_1): now also J2.33 (Pin_33)
- net at GNDREGLE1.1 (Pin_1), J1.22: now also J2.35 (Pin_35)
- net at J1.10, PT100Blanc1.1 (Pin_1): now also J2.37 (Pin_37)
- net at J1.23, TOPZEROREGLE1.1 (Pin_1): now also J2.39 (Pin_39)
- net at J1.11, PT100Blanc2.1 (Pin_1): now also J2.41 (Pin_41)
- net at B+REGLE1.1 (Pin_1), J1.24: now also J2.43 (Pin_43)
- net at J1.12, PT100Rouge1.1 (Pin_1): now also J2.45 (Pin_45)
- net at A+REGLE1.1 (Pin_1), J1.25: now also J2.47 (Pin_47)
- net at J1.13, PT100Rouge2.1 (Pin_1): now also J2.49 (Pin_49)
- net at J1.2, Terre2.1 (Pin_1): now also J2.5 (Pin_5)
- net at IFC-1.1 (Pin_1), J1.15: now also J2.7 (Pin_7)
- net at J1.3, VMoteur1.1 (Pin_1): now also J2.9 (Pin_9)
- new net: J2.2 (Pin_2), J4.1
- new net: J2.38 (Pin_38), J4.10
- new net: J2.42 (Pin_42), J4.11
- new net: J2.46 (Pin_46), J4.12
- new net: J2.50 (Pin_50), J4.13
- new net: J2.4 (Pin_4), J4.14
- new net: J2.8 (Pin_8), J4.15
- new net: J2.12 (Pin_12), J4.16
- new net: J2.16 (Pin_16), J4.17
- new net: J2.20 (Pin_20), J4.18
- new net: J2.24 (Pin_24), J3.2 (Pin_2), J4.19
- new net: J2.6 (Pin_6), J4.2
- new net: J2.28 (Pin_28), J3.3 (Pin_3), J4.20
- new net: J2.32 (Pin_32), J3.4 (Pin_4), J4.21
- new net: J2.36 (Pin_36), J3.5 (Pin_5), J4.22
- new net: J2.40 (Pin_40), J4.23
- new net: J2.44 (Pin_44), J4.24
- new net: J2.48 (Pin_48), J4.25
- new net: J2.10 (Pin_10), J4.3
- new net: J2.14 (Pin_14), J4.4
- new net: J2.18 (Pin_18), J4.5
- new net: J2.22 (Pin22), J4.6
- new net: J2.26 (Pin_26), J4.7
- new net: J2.30 (Pin_30), J4.8
- new net: J2.34 (Pin_34), J3.1 (Pin_1), J4.9
- new net gnd: J1.26, J1.27, J4.26, J4.27
