File: LI600 SWITCH.kicad_pcb (KiCad board)
At the start: 2 copper layers, 68 x 67 mm, 29 parts, among them J1 5443991, J2 Conn_02x25_Odd_Even, J3 Conn_01x05_P2.54mm_pinheader_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, J4 5443991

Commit message: version finale 19/12/2024
Signed-off-by: TEST-BANC <TEST-BANC@DOMOMICRON.LOCAL>
Parts:
- moved TOPZEROREGLE1 12.9 mm to (158.3, 103.9)
- moved SwitchOptique1 12.7 mm to (158.3, 91.6)
- moved IDC-1+IFC-1 8.31 mm to (155.7, 75.8)
- moved GNDREGLE1 7.90 mm to (158.2, 101.6)
- moved SwitchOptique2 7.20 mm to (158.2, 94.4)
- moved +5VREGLE1 3.20 mm to (158.2, 99.3)
- moved J3 2.24 mm to (163.2, 91.6)
- moved SwitchOptique3 1.90 mm to (158.2, 96.8)
Routing:
- net Net-(J2-Pin_23): track 42.8 -> 32.3 mm
- net Net-(B+REGLE1-Pin_1): track 75.4 -> 65.0 mm
- net Net-(J2-Pin_39): track 57.7 -> 48.1 mm, vias 0 -> 1
- net Net-(A+REGLE1-Pin_1): track 81.5 -> 72.8 mm
- net Net-(GNDREGLE1-Pin_1): track 50.0 -> 44.1 mm, vias 0 -> 2
- net Net-(J2-Pin_45): track 64.4 -> 60.1 mm
- net Net-(J2-Pin_41): track 52.7 -> 48.7 mm
- net Net-(J2-Pin_37): track 50.0 -> 46.3 mm
- net Net-(GNDMoteur2-Pin_1): track 45.0 -> 42.0 mm
- net Net-(J2-Pin_9): track 56.3 -> 53.3 mm
- net Net-(J2-Pin_49): track 65.5 -> 62.6 mm
- net Net-(GNDMoteur1-Pin_1): track 40.5 -> 37.8 mm, vias 1 -> 0
- net Net-(J2-Pin_1): track 72.0 -> 69.6 mm
- net Net-(J2-Pin_34): track 27.7 -> 30.1 mm
- net Net-(J2-Pin_33): track 41.1 -> 39.1 mm
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